File: MemoryDMABoard/Schematic/MemoryDMABoard.sch (KiCad schematic (older format))
At the start: 120 parts, among them J1 Bus_ISA_8bit, U1 74LS244, U10 74LS257, U11 74LS244, U13 8237, U14 74LS373, U15 74LS245, U16 74LS125, U17 74LS245, U18 74LS670, U19 MCM6665, U2 74LS04, U20 MCM6665, U21 MCM6665, U22 MCM6665, U23 MCM6665, U24 MCM6665, U25 MCM6665, U26 MCM6665, U27 MCM6665, U28 MCM6665, U29 MCM6665, U30 MCM6665, U31 MCM6665, U32 MCM6665, U33 MCM6665, U34 MCM6665, U35 MCM6665, U36 MCM6665, U37 MCM6665, U38 MCM6665, U39 MCM6665, U40 MCM6665, U41 MCM6665, U42 MCM6665, U43 MCM6665, U44 MCM6665, U45 MCM6665, U46 MCM6665, U47 MCM6665, U48 MCM6665, U49 MCM6665, U5 82S153, U50 MCM6665, U6 74LS257, U7 74LS244, U8 74LS260, U9 82S153

Commit message: First pass of MemoryDMABoard schematic complete.
Parts:
- added R4: 2K2, symbol Device:R
- added U12, U4: 74LS74, symbol 74xx:74LS74
- added unit 4 of U2
- added unit 5 of U2
- added unit 1 of U3
- added unit 5 of U3
- added U51: 74LS00, symbol 74xx:74LS00
- gave numbers to parts that had none: 1
Connections:
- net +5V: now also J1.29 (VCC), R4.2, U12.14 (VCC), U3.14 (VCC), U4.14 (VCC), U51.14 (VCC)
- net BRDY: now also U12.12 (D), U51.9
- net DMACLK: now also U12.11 (C), U12.3 (C)
- net GND: now also U12.7 (GND), U3.7 (GND), U4.7 (GND), U51.7 (GND)
- net HSCLK: now also U4.11 (C), U4.3 (C)
- net SRDY: now also U12.6 (~Q)
- net ~AMUX: now also U3.5, U5.19 (B9)
- net ~IR: now also U51.1
- net ~IW: now also U51.2
- net ~MR: now also U2.11
- net ~MW: now also U2.9
- net at U5.8 (I7): now also U4.9 (Q)
- net at U5.9 (B0): now also U4.12 (D), U4.5 (Q)
- new net: U51.4, U51.5
- new net: U51.10, U51.11
- new net: U12.2 (D), U51.8
- new net: U12.8 (~Q), U51.13
- new net _2K2_PULLUP: R4.1, U12.1 (~R), U12.10 (~S), U12.4 (~S), U4.10 (~S), U4.2 (D), U4.4 (~S)
- new net _IR_OR_IW: U12.13 (~R), U51.12, U51.3
- new net _MR: U2.10, U3.1
- new net _MR_OR_MW: U3.3, U4.1 (~R), U4.13 (~R)
- new net _MW: U2.8, U3.2
- no-connect marks 44 -> 49
Other:
- note added: "8237 DMA CONTROLLER"
- note added: "8237 READY TIMING"
- note added: "ADDRESS DECODING"
- note added: "BI-DIRECTIONAL BUS BUFFERING AND ADDRESS LINE DRIVING"
- note added: "DECOUPLING\n(TANDY SCHEMATIC\nSHEET 1)"
- note added: "DRAM CONTROL LOGIC/TIMING"
- note added: "DRAM MULTIPLEXING"
- note added: "DRAM SECTION (TANDY SCHEMATIC SHEET 2)"
- note added: "JUMPER CONFIGURATION"
- note added: "MISCELLANEOUS"
- note added: "MISCELLANEOUS POWER"
- note added: "On a real board, these inputs \ndo appear to be connected \nand otherwise floating."
- note added: "The Tandy schematic shows this\noutput driving HSCLK which makes \nno sense. Checking a real board,\nit appears to be not connected"
- note added: "UNI-DIRECTIONAL\nBUS BUFFERING"
- note removed: "BUS Buffering"
- note removed: "DRAM SECTION (Tandy Schematic Sheet 2)"
- moved on the sheet: C1, C10, C11, C12, C13, C14, C15, C16, C17, C18, C19, C2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
