File: MemoryDMABoard/Schematic/MemoryDMABoard.sch (KiCad schematic (older format))
At the start: 124 parts, among them J1 Bus_ISA_8bit, U1 74LS244, U10 74LS257, U11 74LS244, U12 74LS74, U13 8237, U14 74LS373, U15 74LS245, U16 74LS125, U17 74LS245, U18 74LS670, U19 MCM6665, U2 74LS04, U20 MCM6665, U21 MCM6665, U22 MCM6665, U23 MCM6665, U24 MCM6665, U25 MCM6665, U26 MCM6665, U27 MCM6665, U28 MCM6665, U29 MCM6665, U3 74LS32, U30 MCM6665, U31 MCM6665, U32 MCM6665, U33 MCM6665, U34 MCM6665, U35 MCM6665, U36 MCM6665, U37 MCM6665, U38 MCM6665, U39 MCM6665, U4 74LS74, U40 MCM6665, U41 MCM6665, U42 MCM6665, U43 MCM6665, U44 MCM6665, U45 MCM6665, U46 MCM6665, U47 MCM6665, U48 MCM6665, U49 MCM6665, U5 82S153, U50 MCM6665, U51 74LS00, U6 74LS257, U7 74LS244, U8 74LS260, U9 82S153

Commit message: Minor text change to MemoryDMABoard schematic.
Other:
- note added: "BIDIRECTIONAL BUS BUFFERING AND ADDRESS LINE DRIVING"
- note added: "UNIDIRECTIONAL\nBUS BUFFERING"
- note removed: "BI-DIRECTIONAL BUS BUFFERING AND ADDRESS LINE DRIVING"
- note removed: "UNI-DIRECTIONAL\nBUS BUFFERING"
Changed lines of the file:
@@
 	17600 7350 17600 600
 Text Notes 17700 950  0    79   ~ 0
-UNI-DIRECTIONAL\nBUS BUFFERING
+UNIDIRECTIONAL\nBUS BUFFERING
 Text Notes 17850 7650 0    79   ~ 0
-BI-DIRECTIONAL BUS BUFFERING AND ADDRESS LINE DRIVING
+BIDIRECTIONAL BUS BUFFERING AND ADDRESS LINE DRIVING
 Wire Notes Line
 	22750 7450 17600 7450
